Commit message: feat: end effector meshes included

File: gripper_description/urdf/measurement_tool.xacro (robot description, xacro)
@@ -16,5 +16,6 @@
           <!-- The path to the visual meshes in the package. -->
           <!-- <mesh filename="package://ur5_with_measurement_tool/meshes/visual/measurement_tool.stl"/> -->
-          <cylinder length="0.6" radius="0.3"/>
+          <mesh filename="package://ur_haptics_teleop_ros/gripper_description/meshes/ee.stl"/>
+          <!-- <cylinder length="0.6" radius="0.3"/>  -->
         </geometry>
       </visual>
